Commit message: 2d lidarを取り付け、scanトピックが確認できるところまで完了。rvizで出力も見れている。

File: src/ugv_sim/hunter_se/hunter_se_description/urdf/hunter_se_description.xacro (robot description, xacro)
@@ -369,3 +369,34 @@
       xyz="0 0 1" />
   </joint>
+  <!-- MID-360 LiDAR Sensor -->
+  <link name="mid360_link">
+    <inertial>
+      <origin xyz="0 0 0" rpy="0 0 0"/>
+      <mass value="0.1"/>
+      <inertia
+        ixx="0.001" ixy="0" ixz="0"
+        iyy="0.001" iyz="0"
+        izz="0.001"/>
+    </inertial>
+    <visual>
+      <origin xyz="0 0 0" rpy="0 0 0"/>
+      <geometry>
+        <cylinder radius="0.05" length="0.08"/>
+      </geometry>
+      <material name="mid360_material">
+        <color rgba="0.2 0.2 0.2 1"/>
+      </material>
+    </visual>
+    <collision>
+      <origin xyz="0 0 0" rpy="0 0 0"/>
+      <geometry>
+        <cylinder radius="0.05" length="0.08"/>
+      </geometry>
+    </collision>
+  </link>
+  <joint name="mid360_joint" type="fixed">
+    <origin xyz="0 0 0.15" rpy="0 0 0"/>
+    <parent link="base_link"/>
+    <child link="mid360_link"/>
+  </joint>
 </robot>

File: src/ugv_sim/hunter_se/hunter_se_gazebo/xacro/hunter_se_gazebo.xacro (robot description, xacro)
@@ -483,4 +483,35 @@
     <axis
       xyz="0 0 1" />
+  </joint>
+  <!-- MID-360 LiDAR Sensor -->
+  <link name="mid360_link">
+    <inertial>
+      <origin xyz="0 0 0" rpy="0 0 0"/>
+      <mass value="0.1"/>
+      <inertia
+        ixx="0.001" ixy="0" ixz="0"
+        iyy="0.001" iyz="0"
+        izz="0.001"/>
+    </inertial>
+    <visual>
+      <origin xyz="0 0 0" rpy="0 0 0"/>
+      <geometry>
+        <cylinder radius="0.05" length="0.08"/>
+      </geometry>
+      <material name="mid360_material">
+        <color rgba="0.2 0.2 0.2 1"/>
+      </material>
+    </visual>
+    <collision>
+      <origin xyz="0 0 0" rpy="0 0 0"/>
+      <geometry>
+        <cylinder radius="0.05" length="0.08"/>
+      </geometry>
+    </collision>
+  </link>
+  <joint name="mid360_joint" type="fixed">
+    <origin xyz="0 0 0.15" rpy="0 0 0"/>
+    <parent link="base_link"/>
+    <child link="mid360_link"/>
   </joint>
 <xacro:macro name="wheel_transmission" params="name">
